File: cheap_ass_robot.kicad_pcb (KiCad board)
At the start: 2 copper layers, 68.6 x 53.3 mm, 49 parts, among them IC1 MC34063A, IC2 ATMEGA328P-AU-R, IC3 FT232RL, IC4 L293DD, J1 USB_B, J2 DIGITAL 2, J3 ANALOG IN, J4 POWER, J5 DIGITAL 1, M1 Motor_DC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

Commit message: all out war against heat
Parts:
- added L2: L, Inductors_SMD:L_0805, F.Cu at (141.0, 106.7)
- added L3: L, Inductors_SMD:L_0805, F.Cu at (136.5, 106.7)
- moved D1 14.2 mm to (129.5, 88.9)
- moved R3 13.1 mm to (123.2, 89.5)
- moved D2 5.68 mm to (132.1, 104.1), turned to 180 degrees
- moved L1 1.91 mm to (145.4, 106.7)
- moved D3 1.80 mm to (123.2, 86.4)
- moved SW1 1.27 mm to (120.7, 97.8)
- moved F1 1.27 mm to (123.2, 82.5)
Connections:
- IC2 pad 19: Net-(IC2-Pad19) -> (no net)
- IC2 pad 22: Net-(IC2-Pad22) -> (no net)
- IC3 pad 10: Net-(IC3-Pad10) -> (no net)
- IC3 pad 11: Net-(IC3-Pad11) -> (no net)
- IC3 pad 12: Net-(IC3-Pad12) -> (no net)
- IC3 pad 13: Net-(IC3-Pad13) -> (no net)
- IC3 pad 14: Net-(IC3-Pad14) -> (no net)
- IC3 pad 19: Net-(IC3-Pad19) -> (no net)
- IC3 pad 24: Net-(IC3-Pad24) -> (no net)
- IC3 pad 27: Net-(IC3-Pad27) -> (no net)
- IC3 pad 28: Net-(IC3-Pad28) -> (no net)
- IC3 pad 3: Net-(IC3-Pad3) -> (no net)
- IC3 pad 6: Net-(IC3-Pad6) -> (no net)
- IC3 pad 8: Net-(IC3-Pad8) -> (no net)
- IC3 pad 9: Net-(IC3-Pad9) -> (no net)
- J2 pad 2: Net-(J2-Pad2) -> (no net)
- J2 pad 3: Net-(J2-Pad3) -> (no net)
- J2 pad 4: Net-(J2-Pad4) -> (no net)
- J4 pad 8: Net-(J4-Pad8) -> (no net)
- J5 pad 4: Net-(J5-Pad4) -> (no net)
- L1 pad 1: Net-(D2-Pad2) -> Net-(L1-Pad1)
Routing:
- net Net-(C1-Pad1): track 48.2 -> 52.5 mm, vias 0 -> 2
- net Net-(D2-Pad2): track 23.2 -> 19.0 mm, vias 0 -> 2
- net Net-(L2-Pad1): track 0.00 -> 2.55 mm
- net Net-(L1-Pad1): track 0.00 -> 2.55 mm
- net Net-(C10-Pad1): track 38.8 -> 36.4 mm
- net Net-(D1-Pad2): track 3.03 -> 4.56 mm
- net Net-(C3-Pad1): track 41.3 -> 42.8 mm
- net Net-(IC1-Pad7): track 28.7 -> 27.8 mm
- net Net-(F1-Pad1): track 8.22 -> 8.82 mm
- net Net-(C2-Pad2): track 39.0 -> 39.3 mm, vias 0 -> 2
Other:
- board text added: "Griffith Cybernetics Cheap Ass Robot Rev. Alpha-3 2019-05-10"
- board text removed: "Griffith Cybernetics Cheap Ass Robot Rev. Alpha-2 2019-04-15"
